File: BatteryModule.kicad_pcb (KiCad board)
At the start: 2 copper layers, 88.8 x 30 mm, 37 parts, among them J1 USB_B_Micro, J2 Conn_01x06, J3 Conn_01x02, J4 Conn_01x02, Q1 Q_NMOS_DSG, Q2 Q_NMOS_DSG, U1 MCP73834T-FCI/UN, U2 AP7215-33YG-13, U2 AP9101CAK6-ANTRG1, U3 AP9101CAK6-ANTRG1

Commit message: Basic layout done
Parts:
- added J1: USB_B_Micro, 12V-SmartSwitch:USB_Micro-B_Amphenol_10118194-0001LF_Horizontal, F.Cu at (-35.6, 272.3)
- added J2: Conn_02x20_Odd_Even, Connector_PinHeader_2.54mm:PinHeader_2x20_P2.54mm_Vertical, F.Cu at (-81.7, 249.9)
- added J4: Conn_01x02_Male, Connector_PinHeader_2.54mm:PinHeader_1x02_P2.54mm_Vertical, F.Cu at (-27.4, 259.5)
- added J5: Conn_01x06, Connector_PinHeader_2.54mm:PinHeader_1x06_P2.54mm_Vertical, B.Cu at (-81.7, 202.5)
- added REF**: 1.152mmHole, SwitchPanel:1.152mmHole, F.Cu at (-84.5, 273.9)
- added REF**: MountingHole_2.7mm_M2.5_DIN965, MountingHole:MountingHole_2.7mm_M2.5_DIN965, F.Cu at (-86.7, 271.7)
- added REF**: MountingHole_2.7mm_M2.5_DIN965, MountingHole:MountingHole_2.7mm_M2.5_DIN965, F.Cu at (-28.7, 271.7)
- added REF**: MountingHole_2.7mm_M2.5_DIN965, MountingHole:MountingHole_2.7mm_M2.5_DIN965, F.Cu at (-28.7, 248.7)
- added REF**: MountingHole_2.7mm_M2.5_DIN965, MountingHole:MountingHole_2.7mm_M2.5_DIN965, F.Cu at (-86.7, 248.7)
- moved JP1 49.1 mm to (-48.5, 208.0)
- moved JP2 21.5 mm to (-80.7, 209.5), turned to 180 degrees
- moved R5 20.5 mm to (-58.0, 203.5), turned to 270 degrees
- moved D3 6.60 mm to (-34.3, 203.4), turned to 270 degrees
- moved R4 6.60 mm to (-34.3, 203.5), turned to 270 degrees
- moved TH1 5.14 mm to (-75.3, 218.3)
- moved J1 3.89 mm to (-35.7, 227.4)
- moved R2 2.70 mm to (-38.7, 203.5), turned to 270 degrees
- moved D2 2.51 mm to (-43.0, 203.5), turned to 270 degrees
- moved D1 2.50 mm to (-38.6, 203.5), turned to 270 degrees
- moved R3 2.50 mm to (-43.0, 203.5), turned to 270 degrees
- moved R1 0.53 mm to (-31.0, 210.0)
- turned R6 to 270 degrees
- turned R7 to 270 degrees
Routing:
- net Net-(C1-Pad1): track 0.00 -> 88.6 mm, vias 0 -> 2
- net P-: track 0.00 -> 64.8 mm, vias 0 -> 2
- net BATT+: track 0.00 -> 62.9 mm, vias 0 -> 2
- net PG: track 0.00 -> 48.8 mm, vias 0 -> 1
- net S1: track 0.00 -> 48.7 mm
- net S2: track 0.00 -> 40.2 mm, vias 0 -> 1
- net Net-(C3-Pad1): track 0.00 -> 37.1 mm
- net (no net): track 0.00 -> 34.9 mm, vias 0 -> 3
- net Net-(Q2-Pad3): track 0.00 -> 29.0 mm, vias 0 -> 2
- net Net-(R9-Pad1): track 0.00 -> 18.9 mm, vias 0 -> 2
- net Net-(Q1-Pad3): track 0.00 -> 18.7 mm, vias 0 -> 3
- net GND: track 0.00 -> 17.3 mm, vias 0 -> 10
- net Net-(D1-Pad2): track 0.00 -> 15.1 mm, vias 0 -> 1
- net +3V3: track 0.00 -> 14.4 mm, vias 0 -> 3
- net Net-(J2-Pad1): track 0.00 -> 9.71 mm
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Other:
- board size 88.8 x 30 mm -> 88.8 x 74.9 mm
- board text added: "39"
- board text added: "3v3"
- board text added: "ESP32-ZIP"
- board text added: "RevB"
- board text added: "SD1"
- board text added: "Vin+"
- board text added: "http://vintlabs.com"
