File: BatteryModule.sch (KiCad schematic (older format))
At the start: 31 parts, among them J1 USB_B_Micro, J2 Conn_01x06, J3 Conn_01x02, J4 Conn_01x02, Q1 Q_NMOS_DSG, Q2 Q_NMOS_DSG, U1 MCP73834T-FCI/UN, U2 AP7215-33YG-13, U3 AP9101CAK6-ANTRG1

Commit message: Basic layout done
Parts:
- added J5: Conn_01x06, Connector_PinHeader_2.54mm:PinHeader_1x06_P2.54mm_Vertical, symbol Connector_Generic:Conn_01x06
Connections:
- net GND: now also J5.3 (Pin_3)
- net at J2.1 (Pin_1), JP2.2 (B): now also J5.1 (Pin_1), J5.2 (Pin_2)
Changed lines of the file:
@@
 	8450 1950 8600 1950
 Wire Wire Line
-	8900 1950 9150 1950
+	8900 1950 9050 1950
+$Comp
+L Connector_Generic:Conn_01x06 J5
+U 1 1 5E1E3E88
+P 10200 2150
+F 0 "J5" H 10280 2142 50  0000 L CNN
+F 1 "Conn_01x06" H 10280 2051 50  0000 L CNN
+F 2 "Connector_PinHeader_2.54mm:PinHeader_1x06_P2.54mm_Vertical" H 10200 2150 50  0001 C CNN
+F 3 "~" H 10200 2150 50  0001 C CNN
+	1    10200 2150
+	1    0    0    -1
+$EndComp
+Wire Wire Line
+	10000 2050 10000 1950
+Wire Wire Line
+	10000 1950 10000 1650
+Connection ~ 10000 1950
+$Comp
+L power:GND #PWR0120
+U 1 1 5E1E93A9
+P 9900 2500
+F 0 "#PWR0120" H 9900 2250 50  0001 C CNN
+F 1 "GND" H 9905 2327 50  0000 C CNN
+F 2 "" H 9900 2500 50  0001 C CNN
+F 3 "" H 9900 2500 50  0001 C CNN
+	1    9900 2500
+	1    0    0    -1
+$EndComp
+Wire Wire Line
+	10000 2150 9900 2150
+Wire Wire Line
+	9900 2150 9900 2500
+Wire Wire Line
+	10000 1650 9050 1650
+Wire Wire Line
+	9050 1650 9050 1950
+Connection ~ 9050 1950
+Wire Wire Line
+	9050 1950 9150 1950
 $EndSCHEMATC
